File: cca/audio_only_cca/audio_only.kicad_pcb (KiCad board)
At the start: 2 copper layers, 76.2 x 50.8 mm, 32 parts, among them J1 CP-43514-ND, P1 CONN_01X04, P2 CONN_01X05, P3 CONN_01X02, P5 CONN_01X03, U5 TLV2362

Commit message: fix: footprint for 1x5 connector
Parts:
- removed P5: CONN_01X03, Socket_Strips:Socket_Strip_Angled_1x03
- added P4: TCONN_01X03, t_footprints:Socket_Strip_Angled_1x03, F.Cu at (99.1, 60.3)
- P1: value CONN_01X04 -> TCONN_01X04; footprint Socket_Strips:Socket_Strip_Angled_1x04 -> t_footprints:Socket_Strip_Angled_1x04
- P2: value CONN_01X05 -> TCONN_01X05; footprint Socket_Strips:Socket_Strip_Angled_1x05 -> t_footprints:Socket_Strip_Angled_1x05
- P3: value CONN_01X02 -> TCONN_01X02

Commit message: Built and fabbed the audio board. It mostly works except for audio on/off changes causes popping only on the right channel.
Parts:
- added REF**: Test_Point_Keystone_5015_Micro-Minature, custom:dummypad, B.Cu at (35.3, 75.3)
- added REF**: Test_Point_Keystone_5015_Micro-Minature, custom:dummypad, B.Cu at (31.9, 75.3)
- added REF**: Test_Point_Keystone_5015_Micro-Minature, custom:dummypad, B.Cu at (27.3, 26.5)
- added REF**: Test_Point_Keystone_5015_Micro-Minature, custom:dummypad, B.Cu at (50.7, 26.5)
Routing:
- net GND: track 0.00 -> 27.7 mm
Other:
- rule trace_min: 0.2 -> 0.5
Changed lines of the file:
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@@
 (kicad_pcb (version 4) (host pcbnew 4.0.5)
   (general
-    (links 51)
+    (links 55)
     (no_connects 0)
-    (area 16.794999 23.253333 110.205001 78.901667)
+    (area 10.784998 22.998 110.205001 78.956)
     (thickness 1.6)
     (drawings 4)
-    (tracks 144)
+    (tracks 151)
     (zones 0)
-    (modules 32)
+    (modules 36)
     (nets 27)
   )
@@
     (last_trace_width 0.5)
     (trace_clearance 0.52)
-    (zone_clearance 0.508)
+    (zone_clearance 0.53)
     (zone_45_only no)
-    (trace_min 0.2)
+    (trace_min 0.5)
     (segment_width 0.2)
     (edge_width 0.15)
@@
     (mod_text_size 1 1)
     (mod_text_width 0.15)
-    (pad_size 1.524 1.524)
-    (pad_drill 0.762)
+    (pad_size 0.5 0.5)
+    (pad_drill 0)
     (pad_to_mask_clearance 0.2)
     (aux_axis_origin 0 0)
     (visible_elements FFFFEF7F)
     (pcbplotparams
-      (layerselection 0x00000_80000001)
+      (layerselection 0x00000_80000000)
       (usegerberextensions false)
       (excludeedgelayer true)
@@
     (add_net "Net-(R13-Pad1)")
   )
+  (module custom:dummypad (layer B.Cu)
+    (at 35.306 75.311)
+    (descr "SMT Test Point- Micro Miniature 5015, http://www.keyelco.com/product-pdf.cfm?p=1353")
+    (tags "Test Point")
+    (attr virtual)
+    (fp_text reference REF** (at 0 2.25) (layer B.SilkS) hide
+      (effects (font (size 1 1) (thickness 0.15)) (justify mirror))
+    )
+    (fp_text value Test_Point_Keystone_5015_Micro-Minature (at 0 -2.25) (layer B.Fab) hide
+      (effects (font (size 1 1) (thickness 0.15)) (justify mirror))
+    )
+    (pad 1 smd rect (at 0 0) (size 0.5 0.5) (layers B.Cu)
+      (net 10 GND) (zone_connect 2))
+  )
+  (module custom:dummypad (layer B.Cu)
+    (at 31.877 75.311)
+    (descr "SMT Test Point- Micro Miniature 5015, http://www.keyelco.com/product-pdf.cfm?p=1353")
+    (tags "Test Point")
+    (attr virtual)
+    (fp_text reference REF** (at 0 2.25) (layer B.SilkS) hide
+      (effects (font (size 1 1) (thickness 0.15)) (justify mirror))
+    )
+    (fp_text value Test_Point_Keystone_5015_Micro-Minature (at 0 -2.25) (layer B.Fab) hide
+      (effects (font (size 1 1) (thickness 0.15)) (justify mirror))
+    )
+    (pad 1 smd rect (at 0 0) (size 0.5 0.5) (layers B.Cu)
+      (net 10 GND) (zone_connect 2))
+  )
+  (module custom:dummypad (layer B.Cu)
+    (at 27.305 26.543)
+    (descr "SMT Test Point- Micro Miniature 5015, http://www.keyelco.com/product-pdf.cfm?p=1353")
+    (tags "Test Point")
+    (attr virtual)
+    (fp_text reference REF** (at 0 2.25) (layer B.SilkS) hide
+      (effects (font (size 1 1) (thickness 0.15)) (justify mirror))
+    )
+    (fp_text value Test_Point_Keystone_5015_Micro-Minature (at 0 -2.25) (layer B.Fab) hide
+      (effects (font (size 1 1) (thickness 0.15)) (justify mirror))
+    )
+    (pad 1 smd rect (at 0 0) (size 0.5 0.5) (layers B.Cu)
+      (net 10 GND) (zone_connect 2))
+  )
   (module t_footprints:C_Radial_D5_L12_P2 (layer F.Cu)
     (at 65.945 35.56)
@@
       (rotate (xyz 0 0 180))
     )
+  )
+  (module custom:dummypad (layer B.Cu)
+    (at 50.673 26.543)
+    (descr "SMT Test Point- Micro Miniature 5015, http://www.keyelco.com/product-pdf.cfm?p=1353")
+    (tags "Test Point")
+    (attr virtual)
+    (fp_text reference REF** (at 0 2.25) (layer B.SilkS) hide
+      (effects (font (size 1 1) (thickness 0.15)) (justify mirror))
+    )
+    (fp_text value Test_Point_Keystone_5015_Micro-Minature (at 0 -2.25) (layer B.Fab) hide
+      (effects (font (size 1 1) (thickness 0.15)) (justify mirror))
+    )
+    (pad 1 smd rect (at 0 0) (size 0.5 0.5) (layers B.Cu)
+      (net 10 GND) (zone_connect 2))
   )
   (gr_line (start 25.4 76.2) (end 25.4 25.4) (layer Edge.Cuts) (width 0.15))
@@
   (segment (start 61.595 49.53) (end 58.42 49.53) (width 0.5) (layer B.Cu) (net 9))
   (segment (start 58.42 49.53) (end 55.245 52.705) (width 0.5) (layer B.Cu) (net 9))
+  (segment (start 31.877 75.311) (end 32.3596 75.7936) (width 0.5) (layer B.Cu) (net 10))
+  (segment (start 32.3596 75.7936) (end 34.8234 75.7936) (width 0.5) (layer B.Cu) (net 10))
+  (segment (start 34.8234 75.7936) (end 35.306 75.311) (width 0.5) (layer B.Cu) (net 10))
+  (segment (start 50.673 26.543) (end 50.038 25.908) (width 0.5) (layer B.Cu) (net 10))
+  (segment (start 50.038 25.908) (end 28.69 25.908) (width 0.5) (layer B.Cu) (net 10))
+  (segment (start 28.69 25.908) (end 28.055 26.543) (width 0.5) (layer B.Cu) (net 10))
+  (segment (start 28.055 26.543) (end 27.305 26.543) (width 0.5) (layer B.Cu) (net 10))
   (segment (start 96.52 50.94) (end 96.52 55.3974) (width 0.5) (layer B.Cu) (net 11))
   (segment (start 96.52 55.3974) (end 98.9076 57.785) (width 0.5) (layer B.Cu) (net 11))
@@
   (segment (start 38.815 60.96) (end 27.94 60.96) (width 0.5) (layer B.Cu) (net 26))
   (zone (net 10) (net_name GND) (layer B.Cu) (hatch edge 0.508)
-    (connect_pads (clearance 0.52))
+    (connect_pads (clearance 0.53))
     (min_thickness 0.254)
-    (fill yes (arc_segments 16) (thermal_gap 0.6) (thermal_bridge_width 0.26))
+    (fill yes (arc_segments 32) (thermal_gap 0.6) (thermal_bridge_width 0.26))
     (polygon
       (pts
